File: kicad projects/switchlab.kicad_pcb (KiCad board)
At the start: 2 copper layers, 93.3 x 134.3 mm, 49 parts, among them SW1 SW_Push, SW10 SW_Push, SW11 SW_Push, SW12 SW_Push, SW13 SW_Push, SW14 SW_Push, SW15 SW_Push, SW16 SW_Push, SW17 SW_Push, SW18 SW_Push, SW19 SW_Push, SW2 SW_Push, SW20 SW_Push, SW3 SW_Push, SW4 SW_Push, SW5 SW_Push, SW6 SW_Push, SW7 SW_Push, SW8 SW_Push, SW9 SW_Push, U1 XIAO_ESP32_S3

Commit message: Add files via upload
Parts:
- moved D16 0.64 mm to (130.5, 60.0)
- moved D18 0.64 mm to (130.5, 63.8)
- moved D19 0.64 mm to (141.9, 67.6)
- moved D1 0.64 mm to (120.0, 39.1)
- moved D10 0.64 mm to (127.6, 49.5)
- moved D15 0.64 mm to (120.0, 60.0)
- moved D17 0.64 mm to (120.0, 63.8)
- moved D2 0.64 mm to (123.8, 39.1)
- moved D3 0.64 mm to (127.6, 39.1)
- moved D8 0.64 mm to (120.0, 49.5)
- moved D9 0.64 mm to (123.8, 49.5)
- moved D11 0.63 mm to (131.4, 49.5)
- moved D12 0.63 mm to (135.3, 49.5)
- moved D13 0.63 mm to (139.1, 49.5)
- moved D14 0.63 mm to (142.9, 49.5)
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Connections:
- ? pad 1: (no net) -> bat+ (x2)
- ? pad 2: (no net) -> bat- (x2)
Routing:
- net (no net): track 408.0 -> 0.00 mm, vias 7 -> 0
- net bat-: track 0.00 -> 211.0 mm, vias 0 -> 5
- net bat+: track 0.00 -> 196.9 mm, vias 0 -> 2
- net Net-(D4-A): track 83.3 -> 162.0 mm, vias 0 -> 4
- net Net-(D15-A): track 76.3 -> 147.3 mm, vias 1 -> 8
- net Net-(D2-A): track 70.2 -> 124.2 mm, vias 1 -> 6
- net Net-(D7-A): track 106.3 -> 145.1 mm, vias 2 -> 7
- net Net-(D9-A): track 102.9 -> 135.7 mm, vias 1 -> 2
- net Net-(D10-A): track 122.9 -> 146.7 mm, vias 1 -> 6
- net Net-(D3-A): track 67.6 -> 91.2 mm, vias 0 -> 3
- net Net-(D17-A): track 112.2 -> 134.7 mm, vias 3 -> 4
- net Net-(D6-A): track 67.4 -> 87.7 mm, vias 0 -> 5
- net Net-(D5-A): track 81.3 -> 94.7 mm, vias 1 -> 7
- net Net-(D16-A): track 100.3 -> 111.0 mm, vias 0 -> 2
- net Net-(D11-A): track 116.3 -> 126.7 mm, vias 2 -> 8
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